Commit message: 0625_增加了地形_增加了sim2sim

File: resources/robots/h1_2_description/h1_2.urdf (robot description, URDF)
Before this commit: robot h1_2, 58 links, 57 joints
Links:
- removed link L_hand_base_link
- removed link L_index_intermediate
- removed link L_index_proximal
- removed link L_middle_intermediate
- removed link L_middle_proximal
- removed link L_pinky_intermediate
- removed link L_pinky_proximal
- removed link L_ring_intermediate
- removed link L_ring_proximal
- removed link L_thumb_distal
- removed link L_thumb_intermediate
- removed link L_thumb_proximal
- removed link L_thumb_proximal_base
- removed link R_hand_base_link
- removed link R_index_intermediate
- removed link R_index_proximal
- removed link R_middle_intermediate
- removed link R_middle_proximal
- removed link R_pinky_intermediate
- removed link R_pinky_proximal
- removed link R_ring_intermediate
- removed link R_ring_proximal
- removed link R_thumb_distal
- removed link R_thumb_intermediate
- removed link R_thumb_proximal
- removed link R_thumb_proximal_base
- link left_ankle_roll_link: geometry collision sphere radius=0.005; collision sphere radius=0.005
- link left_elbow_link: geometry collision box size=0.01 0.01 0.01; visual mesh filename=meshes/left_elbow_link.STL
- link left_hip_pitch_link: geometry collision cylinder length=0.02 radius=0.02; visual mesh filename=meshes/left_hip_pitch_link.STL
- link left_hip_roll_link: geometry collision cylinder length=0.2 radius=0.02; visual mesh filename=meshes/left_hip_roll_link.STL
- link left_shoulder_pitch_link: geometry collision box size=0.01 0.01 0.01; visual mesh filename=meshes/left_shoulder_pitch_link.STL
- link left_shoulder_roll_link: geometry collision box size=0.01 0.01 0.01; visual mesh filename=meshes/left_shoulder_roll_link.STL
- link left_shoulder_yaw_link: geometry collision box size=0.01 0.01 0.01; visual mesh filename=meshes/left_shoulder_yaw_link.STL
- link left_wrist_pitch_link: geometry collision box size=0.01 0.01 0.01; visual mesh filename=meshes/left_wrist_pitch_link.STL
- link left_wrist_roll_link: geometry collision box size=0.01 0.01 0.01; visual mesh filename=meshes/left_wrist_roll_link.STL
- link left_wrist_yaw_link: geometry collision box size=0.01 0.01 0.01; visual mesh filename=meshes/wrist_yaw_link.STL
- link right_ankle_roll_link: geometry collision sphere radius=0.005; collision sphere radius=0.005
- link right_elbow_link: geometry collision box size=0.01 0.01 0.01; visual mesh filename=meshes/right_elbow_link.STL
- link right_hip_pitch_link: geometry collision cylinder length=0.02 radius=0.02; visual mesh filename=meshes/right_hip_pitch_link.STL
- link right_hip_roll_link: geometry collision cylinder length=0.2 radius=0.02; visual mesh filename=meshes/right_hip_roll_link.STL
- link right_shoulder_pitch_link: geometry collision box size=0.01 0.01 0.01; visual mesh filename=meshes/right_shoulder_pitch_link.STL
- link right_shoulder_roll_link: geometry collision box size=0.01 0.01 0.01; visual mesh filename=meshes/right_shoulder_roll_link.STL
- link right_shoulder_yaw_link: geometry collision box size=0.01 0.01 0.01; visual mesh filename=meshes/right_shoulder_yaw_link.STL
- link right_wrist_pitch_link: geometry collision box size=0.01 0.01 0.01; visual mesh filename=meshes/right_wrist_pitch_link.STL
- link right_wrist_roll_link: geometry collision box size=0.01 0.01 0.01; visual mesh filename=meshes/right_wrist_roll_link.STL
- link right_wrist_yaw_link: geometry collision box size=0.01 0.01 0.01; visual mesh filename=meshes/wrist_yaw_link.STL
Joints:
- removed joint L_base_link_joint
- removed joint L_index_intermediate_joint
- removed joint L_index_proximal_joint
- removed joint L_middle_intermediate_joint
- removed joint L_middle_proximal_joint
- removed joint L_pinky_intermediate_joint
- removed joint L_pinky_proximal_joint
- removed joint L_ring_intermediate_joint
- removed joint L_ring_proximal_joint
- removed joint L_thumb_distal_joint
- removed joint L_thumb_intermediate_joint
- removed joint L_thumb_proximal_pitch_joint
- removed joint L_thumb_proximal_yaw_joint
- removed joint R_base_link_joint
- removed joint R_index_intermediate_joint
- removed joint R_index_proximal_joint
- removed joint R_middle_intermediate_joint
- removed joint R_middle_proximal_joint
- removed joint R_pinky_intermediate_joint
- removed joint R_pinky_proximal_joint
- removed joint R_ring_intermediate_joint
- removed joint R_ring_proximal_joint
- removed joint R_thumb_distal_joint
- removed joint R_thumb_intermediate_joint
- removed joint R_thumb_proximal_pitch_joint
- removed joint R_thumb_proximal_yaw_joint
